File: Electrical Schematics/Igniter Circuit.kicad_sch (KiCad schematic)
At the start: 8 parts, among them SW1 SW_SPST

Commit message: E-Match Circuit
Other:
- note added: "Igniter"
- note removed: "E-MATCH"
Changed lines of the file:
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@@
 		)
 	)
-	(text "E-MATCH\n"
+	(text "Igniter\n"
 		(exclude_from_sim no)
 		(at 170.18 122.174 0)
