File: Electrical Schematics/EMatch.kicad_sch (KiCad schematic)
At the start: 3 parts, among them U1 34.81-9024

Commit message: Updated schematics.
Parts:
- removed RL2: AZSR131-1AE-12D, Relay_THT:Relay_SPST_Zettler-AZSR131, symbol Relay:AZSR131-1AE-12D
- added K1: DIPxx-1Cxx-51x, Relay_THT:Relay_StandexMeder_DIP_LowProfile, symbol Relay:DIPxx-1Cxx-51x
Connections:
- net Digital OUT is gone; now on net GND: U1.A1
- net +24V: now also K1.14; no longer LA2.1 (-)
- net GND: now also LA2.1 (-), K1.1, K1.2
- net at LA2.2 (+): now also K1.7, K1.8
- net at U1.14: now also K1.6
